File: BAU-Elec/BAU-Elec.kicad_sch (KiCad schematic)
At the start: 18 parts, among them K1 G2RL-1-E, P16NF06L1 P16NF06L, U2 74LS04

Commit message: Fix: missing wires
Connections:
- net primer_button: now also NA555P1.4 (R), R2.2
- net stop_button: now also NA555P1.2 (TR), R1.2
Changed lines of the file:
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@@
+    )
+  )
+  (global_label "stop_button" (shape input) (at 31.75 104.14 180) (fields_autoplaced)
+    (effects (font (size 1.27 1.27)) (justify right))
+    (property "Intersheetrefs" "${INTERSHEET_REFS}" (at 17.698 104.14 0)
+      (effects (font (size 1.27 1.27)) (justify right) hide)
     )
   )
@@
     )
   )
-  (global_label "5V" (shape input) (at 24.13 114.3 180) (fields_autoplaced)
+  (global_label "5V" (shape input) (at 31.75 121.92 270) (fields_autoplaced)
     (effects (font (size 1.27 1.27)) (justify right))
-    (property "Intersheetrefs" "${INTERSHEET_REFS}" (at 18.8467 114.3 0)
+    (property "Intersheetrefs" "${INTERSHEET_REFS}" (at 31.75 127.2033 90)
       (effects (font (size 1.27 1.27)) (justify right) hide)
     )
@@
     )
   )
+  (global_label "primer_button" (shape input) (at 31.75 114.3 180) (fields_autoplaced)
+    (effects (font (size 1.27 1.27)) (justify right))
+    (property "Intersheetrefs" "${INTERSHEET_REFS}" (at 15.6417 114.3 0)
+      (effects (font (size 1.27 1.27)) (justify right) hide)
+    )
+  )
   (global_label "bat_out" (shape input) (at 163.83 36.83 90) (fields_autoplaced)
     (effects (font (size 1.27 1.27)) (justify left))
@@
     )
   )
-  (symbol (lib_id "Device:R") (at 27.94 114.3 90) (unit 1)
+  (symbol (lib_id "Device:R") (at 31.75 118.11 180) (unit 1)
     (in_bom yes) (on_board yes) (dnp no)
-    (property "Reference" "R2" (at 26.67 115.57 0)
+    (property "Reference" "R2" (at 33.02 119.38 0)
       (effects (font (size 1.27 1.27)) (justify left) hide)
     )
-    (property "Value" "10k" (at 27.94 114.3 90)
+    (property "Value" "10k" (at 31.75 118.11 90)
       (effects (font (size 1.27 1.27)))
     )
-    (property "Footprint" "Resistor_THT:R_Axial_DIN0207_L6.3mm_D2.5mm_P7.62mm_Horizontal" (at 27.94 116.078 90)
+    (property "Footprint" "Resistor_THT:R_Axial_DIN0207_L6.3mm_D2.5mm_P7.62mm_Horizontal" (at 33.528 118.11 90)
       (effects (font (size 1.27 1.27)) hide)
     )
-    (property "Datasheet" "~" (at 27.94 114.3 0)
+    (property "Datasheet" "~" (at 31.75 118.11 0)
       (effects (font (size 1.27 1.27)) hide)
     )
