File: PowerBoard-Elec/PowerBoard-Elec.kicad_sch (KiCad schematic)
At the start: 37 parts, among them J1 XT60PW-M, J2 Logique_switch, J3 ADJ_4A, J4 Battery_cells, J5 5V_5A, U1 DCDC_StepDown_Dsun, U10 DCDC_StepDown_XL4015, U11 DCDC_StepDown_MINI560, U12 ADJ_5A, U13 ADJ_5A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

Commit message: Feat: update PowerBoard
Parts:
- removed U6: BAU, CONN_JST_B3P-VH:CONN_JST_B3P-VH, symbol CONN_JST_B3P-VH:B3P-VH_LF__SN_
- added J6: BAU, CONN_JST_B3PS-VH:CONN_JST_B3PS-VH, symbol CONN_JST_B3PS-VH:B3PS-VH
Connections:
- net GND: now also U14.2 (IN-), J6.1; no longer U14.1 (IN+)
- net V_BAT: now also J2.4, J6.2; no longer J2.3
- net V_BAU: now also U14.1 (IN+), J6.3; no longer U14.2 (IN-)
- net V_LOGIQUE: now also J2.2; no longer J2.4
- net at R7.1: now also J2.3; no longer J2.2
- net at J3.1, U4.3 (OUT+): now also R5.1
- net at J3.2, U4.4 (OUT-): no longer R5.1
